Commit message: Add simrad ek transducer

File: urdf/drix_mesh.xacro (robot description, xacro)
@@ -11,3 +11,16 @@
     </visual>
   </link>
+  <link name="${namespace}/ek80">
+    <visual>
+      <geometry>
+        <cylinder length="0.0752" radius="0.06"/>
+      </geometry>
+      <origin rpy="0 1.57075 0" xyz="-0.0376 0 0"/>
+    </visual>
+  </link>
+  <joint name="${namespace}/base_to_ek80" type="fixed">
+      <parent link="${namespace}/base_link"/>
+      <child link="${namespace}/ek80"/>
+      <origin rpy="0 1.57075 0" xyz="-0.728 -0.131 -0.134 " />
+  </joint>
 </robot>

Commit message: Add mbes to tf tree

File: urdf/drix_mesh.xacro (robot description, xacro)
@@ -24,3 +24,16 @@
       <origin rpy="0 1.57075 0" xyz="-0.728 -0.131 -0.134 " />
   </joint>
+  <link name="sonar_vcs">
+    <visual>
+      <geometry>
+        <cylinder length="0.0752" radius="0.06"/>
+      </geometry>
+      <origin rpy="0 1.57075 0" xyz="-0.0376 0 0"/>
+    </visual>
+  </link>
+  <joint name="${namespace}/base_to_sonar_vcs" type="fixed">
+    <parent link="${namespace}/base_link"/>
+    <child link="sonar_vcs"/>
+    <origin rpy="3.14 0 0" xyz="-0.586 0.080 -0.149 " />
+  </joint>
 </robot>

Commit message: Fix mbes frame of reference

File: urdf/drix_mesh.xacro (robot description, xacro)
@@ -32,6 +32,28 @@
     </visual>
   </link>
+  <link name="${namespace}/base_link_north_up">
+    <visual>
+        <geometry>
+            <sphere radius="0.01"/>
+        </geometry>
+    </visual>
+  </link>
+  <joint name="${namespace}/base_north_up_to_base" type="floating">
+    <parent link="${namespace}/base_link_north_up"/>
+    <child link="${namespace}/base_link"/>
+  </joint>
+  <link name="${namespace}/base_link_level">
+    <visual>
+        <geometry>
+            <sphere radius="0.01"/>
+        </geometry>
+    </visual>
+  </link>
+  <joint name="${namespace}/base_north_up_to_base_level" type="floating">
+    <parent link="${namespace}/base_link_north_up"/>
+    <child link="${namespace}/base_link_level"/>
+  </joint>
   <joint name="${namespace}/base_to_sonar_vcs" type="fixed">
-    <parent link="${namespace}/base_link"/>
+    <parent link="${namespace}/base_link_level"/>
     <child link="sonar_vcs"/>
     <origin rpy="3.14 0 0" xyz="-0.586 0.080 -0.149 " />

Commit message: Update ek80 transform

File: urdf/drix_mesh.xacro (robot description, xacro)
@@ -22,5 +22,6 @@
       <parent link="${namespace}/base_link"/>
       <child link="${namespace}/ek80"/>
-      <origin rpy="0 1.57075 0" xyz="-0.728 -0.131 -0.134 " />
+      <!-- <origin rpy="0 1.57075 0" xyz="-0.728 -0.131 -0.134 " /> -->
+      <origin rpy="3.14 0 0" xyz="-0.728 -0.131 -0.134 " />
   </joint>
   <link name="sonar_vcs">
